File: doc/robot diagram/robot diagram.kicad_sch (KiCad schematic)
At the start: 44 parts, among them M1 Motor_DC, M2 Motor_DC, Q1 PMOS, Q2 PMOS, Q3 NMOS, Q4 NMOS, Q5 NMOS, Q6 NMOS, Q7 PMOS, Q8 PMOS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

Commit message: robot diagram
Parts:
- added C6: 1u, symbol Device:C
- added R12: 1k, symbol Device:R
- C1, C3, C5: value C -> 100n
- C2, C4: value C -> 1u
- L1, L2: value L -> 1m
- R1, R4, R7: value R -> 1k
- R10, R9: value R -> 2k
- R11, R3, R6: value R -> 10k
- R2, R5, R8: value R -> 47k
Connections:
- net +5V: now also R12.1
- net GND: now also C6.2
- net PB7: now also C6.1, R12.2
Other:
- moved on the sheet: D3, D4, D5
